File: pcb/cpu.kicad_pcb (KiCad board)
At the start: 2 copper layers, 5 parts

Commit message: wip schematics
Parts:
- removed 74AHC08D.112, 74AHC32D.112, 74HC86D.653: SOIC-14_3.9x8.7mm_P1.27mm, Package_SO:SOIC-14_3.9x8.7mm_P1.27mm
- removed REF** (x2): PinHeader_1x09_P1.00mm_Vertical, Connector_PinHeader_1.00mm:PinHeader_1x09_P1.00mm_Vertical
Routing:
- net (no net): track 281.0 -> 0.00 mm
Other:
- rule pad_to_mask_clearance: 0.051 -> 0
