File: pcb/cpu.sch (KiCad schematic (older format))
At the start: 9 parts, among them J1 Conn_02x16_Counter_Clockwise, J2 Conn_01x16, U1 74LS283, U2 74LS283, U3 74LS283, U4 74LS283

Commit message: wip alu function muxes
Parts:
- added J?: Conn_01x06_MountingPin, symbol Connector_Generic_MountingPin:Conn_01x06_MountingPin
- added U? (x4): mux16, symbol nand2tetris:mux16
- added U? (x16): 74AHCT1G04, symbol 74xGxx:74AHCT1G04
Connections:
- net +5V: now also U4.16 (VCC)
- net GND: now also U?.3 (GND), U?.3 (GND), U?.3 (GND), U?.3 (GND), U?.3 (GND), U?.3 (GND), U?.3 (GND), U?.3 (GND), U?.3 (GND), U?.3 (GND), U?.3 (GND), U?.3 (GND), U?.3 (GND), U?.3 (GND), U?.3 (GND), U?.3 (GND)
- new net VCC: U?.5 (VCC), U?.5 (VCC), U?.5 (VCC), U?.5 (VCC), U?.5 (VCC), U?.5 (VCC), U?.5 (VCC), U?.5 (VCC), U?.5 (VCC), U?.5 (VCC), U?.5 (VCC), U?.5 (VCC), U?.5 (VCC), U?.5 (VCC), U?.5 (VCC), U?.5 (VCC)
- new net f: J?.5 (Pin_5)
- new net no: J?.6 (Pin_6)
- new net nx: J?.2 (Pin_2)
- new net ny: J?.4 (Pin_4), U?.~ (VCC)
- new net opy0: U?.0 (out)
- new net opy1: U?.1 (out)
- new net opy10: U?.10 (out)
- new net opy11: U?.11 (out)
- new net opy12: U?.12 (out)
- new net opy13: U?.13 (out)
- new net opy14: U?.14 (out)
- new net opy15: U?.15 (out)
- new net opy2: U?.2 (out)
- new net opy3: U?.3 (out)
- new net opy4: U?.4 (out)
- new net opy5: U?.5 (out)
- new net opy6: U?.6 (out)
- new net opy7: U?.7 (out)
- new net opy8: U?.8 (out)
- new net opy9: U?.9 (out)
- new net x0: U?.0 (out)
- new net x1: U?.1 (out)
- new net x10: U?.10 (out)
- new net x11: U?.11 (out)
- new net x12: U?.12 (out)
- new net x13: U?.13 (out)
- new net x14: U?.14 (out)
- new net x15: U?.15 (out)
- new net x2: U?.2 (out)
- new net x3: U?.3 (out)
- new net x4: U?.4 (out)
- new net x5: U?.5 (out)
- new net x6: U?.6 (out)
- new net x7: U?.7 (out)
- new net x8: U?.8 (out)
- new net x9: U?.9 (out)
- new net y0: U?.0 (out)
- new net y1: U?.1 (out)
- new net y10: U?.10 (out)
- new net y11: U?.11 (out)
- new net y12: U?.12 (out)
- new net y13: U?.13 (out)
- new net y14: U?.14 (out)
- new net y15: U?.15 (out)
- new net y2: U?.2 (out)
- new net y3: U?.3 (out)
- new net y4: U?.4 (out)
- new net y5: U?.5 (out)
- new net y6: U?.6 (out)
- new net y7: U?.7 (out)
- new net y8: U?.8 (out)
- new net y9: U?.9 (out)
- new net zdy0: U?.0 (out), U?.0 (out), U?.2
- new net zdy1: U?.1 (out), U?.1 (out), U?.2
- new net zdy10: U?.10 (out), U?.10 (out), U?.2
- new net zdy11: U?.11 (out), U?.11 (out), U?.2
- new net zdy12: U?.12 (out), U?.12 (out), U?.2
- new net zdy13: U?.13 (out), U?.13 (out), U?.2
- new net zdy14: U?.14 (out), U?.14 (out), U?.2
- new net zdy15: U?.15 (out), U?.15 (out), U?.2
- new net zdy2: U?.2, U?.2 (out), U?.2 (out)
- new net zdy3: U?.2, U?.3 (out), U?.3 (out)
- new net zdy4: U?.2, U?.4 (out), U?.4 (out)
- new net zdy5: U?.2, U?.5 (out), U?.5 (out)
- new net zdy6: U?.2, U?.6 (out), U?.6 (out)
- new net zdy7: U?.2, U?.7 (out), U?.7 (out)
- new net zdy8: U?.2, U?.8 (out), U?.8 (out)
- new net zdy9: U?.2, U?.9 (out), U?.9 (out)
- new net zx: J?.1 (Pin_1), U?.~ (VCC)
- new net zy: J?.3 (Pin_3), U?.~ (VCC)
Other:
- moved on the sheet: J1, J2, U?A

Commit message: SN74CBT16233 symbol
Parts:
- removed U? (x3): 74LS21, symbol 74xx:74LS21
- removed U? (x3): mux16, symbol nand2tetris:mux16
- removed U? (x16): 74AHCT1G04, symbol 74xGxx:74AHCT1G04
- added U? (x48): 74AHCT1G04, symbol 74xGxx:74AHCT1G04
- added U? (x3): mux16, symbol nand2tetris:mux16
- added U? (x16): 74LS08, symbol 74xx:74LS08
- added U?: SN74CBT16233, symbol nand2tetris:SN74CBT16233
Connections:
- net GND: now also U?.~ (VCC), U?.3 (GND), U?.3 (GND), U?.3 (GND), U?.3 (GND), U?.3 (GND), U?.3 (GND), U?.3 (GND), U?.3 (GND), U?.3 (GND), U?.3 (GND), U?.3 (GND), U?.3 (GND), U?.3 (GND), U?.3 (GND), U?.3 (GND), U?.3 (GND), U?.3 (GND), U?.3 (GND), U?.3 (GND), U?.3 (GND), U?.3 (GND), U?.3 (GND), U?.3 (GND), U?.3 (GND), U?.3 (GND), U?.3 (GND), U?.3 (GND), U?.3 (GND), U?.3 (GND), U?.3 (GND), U?.3 (GND), U?.3 (GND), U?.3 (GND), U?.3 (GND), U?.3 (GND), U?.3 (GND), U?.3 (GND), U?.3 (GND), U?.3 (GND), U?.3 (GND), U?.3 (GND), U?.3 (GND), U?.3 (GND), U?.3 (GND), U?.3 (GND), U?.3 (GND), U?.3 (GND), U?.3 (GND), U?.~ (VCC), U?.~ (VCC), U?.~ (VCC)
- net VCC: now also U?.5 (VCC), U?.5 (VCC), U?.5 (VCC), U?.5 (VCC), U?.5 (VCC), U?.5 (VCC), U?.5 (VCC), U?.5 (VCC), U?.5 (VCC), U?.5 (VCC), U?.5 (VCC), U?.5 (VCC), U?.5 (VCC), U?.5 (VCC), U?.5 (VCC), U?.5 (VCC), U?.5 (VCC), U?.5 (VCC), U?.5 (VCC), U?.5 (VCC), U?.5 (VCC), U?.5 (VCC), U?.5 (VCC), U?.5 (VCC), U?.5 (VCC), U?.5 (VCC), U?.5 (VCC), U?.5 (VCC), U?.5 (VCC), U?.5 (VCC), U?.5 (VCC), U?.5 (VCC), U?.5 (VCC), U?.5 (VCC), U?.5 (VCC), U?.5 (VCC), U?.5 (VCC), U?.5 (VCC), U?.5 (VCC), U?.5 (VCC), U?.5 (VCC), U?.5 (VCC), U?.5 (VCC), U?.5 (VCC), U?.5 (VCC), U?.5 (VCC), U?.5 (VCC), U?.5 (VCC)
- net a0: no longer U1.5 (A1)
- net a1: no longer U1.3 (A2)
- net a10: no longer U3.14 (A3)
- net a11: no longer U3.12 (A4)
- net a12: no longer U4.5 (A1)
- net a13: no longer U4.3 (A2)
- net a14: no longer U4.14 (A3)
- net a15: no longer U4.12 (A4)
- net a2: no longer U1.14 (A3)
- net a3: no longer U1.12 (A4)
- net a4: no longer U2.5 (A1)
- net a5: no longer U2.3 (A2)
- net a6: no longer U2.14 (A3)
- net a7: no longer U2.12 (A4)
- net a8: no longer U3.5 (A1)
- net a9: no longer U3.3 (A2)
- net b0: no longer U1.6 (B1)
- net b1: no longer U1.2 (B2)
- net b10: no longer U3.15 (B3)
- net b11: no longer U3.11 (B4)
- net b12: no longer U4.6 (B1)
- net b13: no longer U4.2 (B2)
- net b14: no longer U4.15 (B3)
- net b15: no longer U4.11 (B4)
- net b2: no longer U1.15 (B3)
- net b3: no longer U1.11 (B4)
- net b4: no longer U2.6 (B1)
- net b5: no longer U2.2 (B2)
- net b6: no longer U2.15 (B3)
- net b7: no longer U2.11 (B4)
- net b8: no longer U3.6 (B1)
- net b9: no longer U3.2 (B2)
- net noty0: now also U?.4
- net noty1: now also U?.4
- net noty10: now also U?.4
- net noty11: now also U?.4
- net noty12: now also U?.4
- net noty13: now also U?.4
- net noty14: now also U?.4
- net noty15: now also U?.4
- net noty2: now also U?.4
- net noty3: now also U?.4
- net noty4: now also U?.4
- net noty5: now also U?.4
- net noty6: now also U?.4
- net noty7: now also U?.4
- net noty8: now also U?.4
- net noty9: now also U?.4
- net nx: now also U?.~ (VCC), U?.~ (VCC)
- net opy0: now also U1.6 (B1), U?.0 (out), U?.1 (1A), U?.2
- net opy1: now also U1.2 (B2), U?.1 (out), U?.2, U?.54 (2A)
- net opy10: now also U3.15 (B3), U?.10 (out), U?.18 (11A), U?.2
- net opy11: now also U3.11 (B4), U?.11 (out), U?.2, U?.37 (12A)
- net opy12: now also U4.6 (B1), U?.12 (out), U?.2, U?.21 (13A)
- net opy13: now also U4.2 (B2), U?.1, U?.13 (out), U?.2, U?.34 (14A)
- net opy14: now also U4.15 (B3), U?.14 (out), U?.2, U?.24 (15A)
- net opy15: now also U4.11 (B4), U?.15 (out), U?.2, U?.31 (16A)
- net opy2: now also U1.15 (B3), U?.2, U?.2 (out), U?.4 (3A)
- net opy3: now also U1.11 (B4), U?.2, U?.3 (out), U?.51 (4A)
- net opy4: now also U2.6 (B1), U?.2, U?.4 (out), U?.7 (5A)
- net opy5: now also U2.2 (B2), U?.2, U?.48 (6A), U?.5 (out)
- net opy6: now also U2.15 (B3), U?.10 (7A), U?.2, U?.6 (out)
- net opy7: now also U2.11 (B4), U?.2, U?.45 (8A), U?.7 (out)
- net opy8: now also U3.6 (B1), U?.15 (9A), U?.2, U?.8 (out)
- net opy9: now also U3.2 (B2), U?.2, U?.40 (10A), U?.9 (out)
- net s0: no longer U1.4 (S1)
- net s1: no longer U1.1 (S2)
- net s10: no longer U3.13 (S3)
- net s11: no longer U3.10 (S4)
- net s12: no longer U4.4 (S1)
- net s13: no longer U4.1 (S2)
- net s14: no longer U4.13 (S3)
- net s15: no longer U4.10 (S4)
- net s2: no longer U1.13 (S3)
- net s3: no longer U1.10 (S4)
- net s4: no longer U2.4 (S1)
- net s5: no longer U2.1 (S2)
- net s6: no longer U2.13 (S3)
- net s7: no longer U2.10 (S4)
- net s8: no longer U3.4 (S1)
- net s9: no longer U3.1 (S2)
- net y0: now also U?.0 (out)
- net y1: now also U?.1 (out)
- net y10: now also U?.10 (out)
- net y11: now also U?.11 (out)
- net y12: now also U?.12 (out)
- net y13: now also U?.13 (out)
- net y14: now also U?.14 (out)
- net y15: now also U?.15 (out)
- net y2: now also U?.2 (out)
- net y3: now also U?.3 (out)
- net y4: now also U?.4 (out)
- net y5: now also U?.5 (out)
- net y6: now also U?.6 (out)
- net y7: now also U?.7 (out)
- net y8: now also U?.8 (out)
- net y9: now also U?.9 (out)
- net zdx0: now also U?.0 (out), U?.0 (out), U?.2
- net zdx1: now also U?.1 (out), U?.1 (out), U?.2
- net zdx10: now also U?.10 (out), U?.10 (out), U?.2
- net zdx11: now also U?.11 (out), U?.11 (out), U?.2
- net zdx12: now also U?.12 (out), U?.12 (out), U?.2
- net zdx13: now also U?.13 (out), U?.13 (out), U?.2
- net zdx14: now also U?.14 (out), U?.14 (out), U?.2
- net zdx15: now also U?.15 (out), U?.15 (out), U?.2
- net zdx2: now also U?.2 (out), U?.2, U?.2 (out)
- net zdx3: now also U?.3 (out), U?.2, U?.3 (out)
- net zdx4: now also U?.4 (out), U?.2, U?.4 (out)
- net zdx5: now also U?.5 (out), U?.2, U?.5 (out)
- net zdx6: now also U?.6 (out), U?.2, U?.6 (out)
- net zdx7: now also U?.7 (out), U?.2, U?.7 (out)
- net zdx8: now also U?.8 (out), U?.2, U?.8 (out)
- net zdx9: now also U?.9 (out), U?.2, U?.9 (out)
- net zdy0: now also U?.0 (out), U?.0 (out), U?.2
- net zdy1: now also U?.1 (out), U?.1 (out), U?.2
- net zdy10: now also U?.10 (out), U?.10 (out), U?.2
- net zdy11: now also U?.11 (out), U?.11 (out), U?.2
- net zdy12: now also U?.12 (out), U?.12 (out), U?.2
- net zdy13: now also U?.13 (out), U?.13 (out), U?.2
- net zdy14: now also U?.14 (out), U?.14 (out), U?.2
- net zdy15: now also U?.15 (out), U?.15 (out), U?.2
- net zdy2: now also U?.2, U?.2 (out), U?.2 (out)
- net zdy3: now also U?.2, U?.3 (out), U?.3 (out)
- net zdy4: now also U?.2, U?.4 (out), U?.4 (out)
- net zdy5: now also U?.2, U?.5 (out), U?.5 (out)
- net zdy6: now also U?.2, U?.6 (out), U?.6 (out)
- net zdy7: now also U?.2, U?.7 (out), U?.7 (out)
- net zdy8: now also U?.2, U?.8 (out), U?.8 (out)
- net zdy9: now also U?.2, U?.9 (out), U?.9 (out)
- net zx: now also U?.~ (VCC)
- new net band0: U?.3
- new net band1: U?.3
- new net band10: U?.3
- new net band11: U?.3
- new net band12: U?.3
- new net band13: U?.3
- new net band14: U?.3
- new net band15: U?.3
- new net band2: U?.3
- new net band3: U?.3
- new net band4: U?.3
- new net band5: U?.3
- new net band6: U?.3
- new net band7: U?.3
- new net band8: U?.3
- new net band9: U?.3
- new net notsum0: U?.4
- new net notsum1: U?.4
- new net notsum10: U?.4
- new net notsum11: U?.4
- new net notsum12: U?.4
- new net notsum13: U?.4
- new net notsum14: U?.4
- new net notsum15: U?.4
- new net notsum2: U?.4
- new net notsum3: U?.4
- new net notsum4: U?.4
- new net notsum5: U?.4
- new net notsum6: U?.4
- new net notsum7: U?.4
- new net notsum8: U?.4
- new net notsum9: U?.4
- new net opx0: U1.5 (A1), U?.0 (out), U?.1
- new net opx1: U1.3 (A2), U?.1, U?.1 (out)
- new net opx10: U3.14 (A3), U?.1, U?.10 (out)
- new net opx11: U3.12 (A4), U?.1, U?.11 (out)
- new net opx12: U4.5 (A1), U?.1, U?.12 (out)
- new net opx13: U4.3 (A2), U?.13 (out)
- new net opx14: U4.14 (A3), U?.1, U?.14 (out)
- new net opx15: U4.12 (A4), U?.1, U?.15 (out)
- new net opx2: U1.14 (A3), U?.1, U?.2 (out)
- new net opx3: U1.12 (A4), U?.1, U?.3 (out)
- new net opx4: U2.5 (A1), U?.1, U?.4 (out)
- new net opx5: U2.3 (A2), U?.1, U?.5 (out)
- new net opx6: U2.14 (A3), U?.1, U?.6 (out)
- new net opx7: U2.12 (A4), U?.1, U?.7 (out)
- new net opx8: U3.5 (A1), U?.1, U?.8 (out)
- new net opx9: U3.3 (A2), U?.1, U?.9 (out)
- new net sum0: U1.4 (S1), U?.2
- new net sum1: U1.1 (S2), U?.2
- new net sum10: U3.13 (S3), U?.2
- new net sum11: U3.10 (S4), U?.2
- new net sum12: U4.4 (S1), U?.2
- new net sum13: U4.1 (S2), U?.2
- new net sum14: U4.13 (S3), U?.2
- new net sum15: U4.10 (S4), U?.2
- new net sum2: U1.13 (S3), U?.2
- new net sum3: U1.10 (S4), U?.2
- new net sum4: U2.4 (S1), U?.2
- new net sum5: U2.1 (S2), U?.2
- new net sum6: U2.13 (S3), U?.2
- new net sum7: U2.10 (S4), U?.2
- new net sum8: U3.4 (S1), U?.2
- new net sum9: U3.1 (S2), U?.2
